Commit message: Simulation Camera and Lidar are working

File: description/robot.urdf.xacro (robot description, xacro)
@@ -3,3 +3,5 @@
 <xacro:include filename="robot_core.xacro" />
 <xacro:include filename="gazebo_control.xacro" />
+<xacro:include filename="lidar.xacro" />
+<xacro:include filename="camera.xacro" />
 </robot>

File: description/robot_core.xacro (robot description, xacro)
@@ -270,70 +270,3 @@
         <material>Gazebo/White</material>
     </gazebo>
-    <!-- Camera Link -->
-    <joint name = "camera_joint" type = "fixed">
-        <parent link = "sensor_tower_link"/>
-        <child link = "camera_link"/>
-        <origin xyz = "${size_item*5/6} 0 0"/>
-    </joint>
-    <link name = "camera_link">
-        <visual>
-            <origin xyz = "${-size_item/6} 0 0"/>
-            <geometry>
-                <box size = "${size_item/3} ${size_item} ${size_item}"/>
-            </geometry>
-            <material name = "orange"/>
-        </visual>
-       <xacro:inertial_box mass="0.025" x="${size_item*2/3}" y="${size_item}" z="${size_item}">
-            <origin xyz= "0 0 0"  rpy="0 0 0"/>
-        </xacro:inertial_box>
-        <visual>
-            <origin xyz = "${size_item/6} 0 0" rpy="0 ${pi/2} 0"/>
-            <geometry>
-                <cylinder radius="${size_item/3}" length = "${size_item/3}"/>
-            </geometry>
-            <material name = "orange"/>
-        </visual>
-        <collision>
-            <geometry>
-                <box size = "${size_item*2/3} ${size_item} ${size_item}"/>
-            </geometry>
-        </collision>
-    </link>
-    <gazebo reference = "camera_link">
-        <material>Gazebo/Orange</material>
-    </gazebo>
-    <!-- Lidar Link -->
-    <joint name = "lidar_joint" type = "fixed">
-        <parent link = "sensor_tower_link"/>
-        <child link = "lidar_link"/>
-        <origin xyz = "${-2*size_item} 0 ${hight_sensor_tower/2}"/>
-    </joint>
-    <link name = "lidar_link">
-        <visual>
-            <origin xyz = "0 0 ${-size_item/4}"/>
-            <geometry>
-                <box size = "${size_item*3} ${size_item*2} ${size_item/2}"/>
-            </geometry>
-            <material name = "green"/>
-        </visual>
-       <xacro:inertial_box mass="0.1" x="${size_item*3}" y="${size_item*2}" z="${size_item*7/6}">
-            <origin xyz= "0 0 ${-size_item/12}"  rpy="0 0 0"/>
-        </xacro:inertial_box>
-        <visual>
-            <origin xyz = "0 0 ${size_item/4}" rpy="0 0 0"/>
-            <geometry>
-                <cylinder radius="${size_item*0.75}" length = "${size_item*2/3}"/>
-            </geometry>
-            <material name = "orange"/>
-        </visual>
-        <collision>
-            <origin xyz= "0 0 ${-size_item/12}"  rpy="0 0 0"/>
-            <geometry>
-                <box size = "${size_item*3} ${size_item*2} ${size_item*7/6}"/>
-            </geometry>
-        </collision>
-    </link>
-    <gazebo reference = "lidar_link">
-        <material>Gazebo/Green</material>
-    </gazebo>
 </robot>
